File: Project/universal vault v2.kicad_sch (KiCad schematic)
At the start: 213 parts, among them J1 USB_C_Receptacle_USB2.0, SW1 RotaryEncoder_Switch, SW2 RotaryEncoder_Switch, SW3 RotaryEncoder_Switch, SW4 SKQGABE010, SW5 RotaryEncoder_Switch, U1 STM32F072CBUx, U2 XC6206PxxxMR, U5 74AHCT1G125

Commit message: version 2 finished, production files created
Connections:
- net rF is gone; now on net rE: SW3.B, U1.16 (PA6)
Other:
- note added: "MCU"
- note added: "PINOUT"
- moved on the sheet: C1, C10, C11, C2, C3, C4, C5, C6, C7, C8, D1, F2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

Commit message: update readme
Connections:
- net rE: no longer SW3.B, U1.16 (PA6)
- new net rF: SW3.B, U1.16 (PA6)
Changed lines of the file:
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@@
     (effects (font (size 1.27 1.27)) (justify left bottom))
   )
-  (label "A7" (at 48.895 62.23 0) (fields_autoplaced)
+  (label "A6" (at 48.895 62.23 0) (fields_autoplaced)
     (effects (font (size 1.27 1.27)) (justify left bottom))
   )

Commit message: changed rgb pin for better software hardware compatibility & fresh production files
Connections:
- net RGB MCU: now also U1.29 (PA8); no longer U1.11 (PA1)
- net col0: now also U1.11 (PA1); no longer U1.10 (PA0)
- net rD: now also U1.28 (PB15); no longer U1.29 (PA8)
Changed lines of the file:
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@@
   (no_connect (at 70.485 85.725))
   (no_connect (at 217.805 74.93))
-  (no_connect (at 70.485 90.805))
   (no_connect (at 70.485 47.625))
+  (no_connect (at 103.505 24.765))
   (no_connect (at 70.485 88.265))
   (no_connect (at 70.485 83.185))
@@
     )
   )
-  (global_label "col0" (shape input) (at 103.505 24.765 0) (fields_autoplaced)
-    (effects (font (size 1.27 1.27)) (justify left))
-    (property "Intersheetrefs" "${INTERSHEET_REFS}" (at 110.5231 24.765 0)
+  (global_label "col0" (shape input) (at 103.505 27.305 0) (fields_autoplaced)
+    (effects (font (size 1.27 1.27)) (justify left))
+    (property "Intersheetrefs" "${INTERSHEET_REFS}" (at 110.5231 27.305 0)
       (effects (font (size 1.27 1.27)) (justify left) hide)
     )
@@
     )
   )
-  (global_label "rD" (shape input) (at 103.505 45.085 0) (fields_autoplaced)
-    (effects (font (size 1.27 1.27)) (justify left))
-    (property "Intersheetrefs" "${INTERSHEET_REFS}" (at 108.467 45.085 0)
-      (effects (font (size 1.27 1.27)) (justify left) hide)
+  (global_label "rD" (shape input) (at 70.485 90.805 180) (fields_autoplaced)
+    (effects (font (size 1.27 1.27)) (justify right))
+    (property "Intersheetrefs" "${INTERSHEET_REFS}" (at 65.523 90.805 0)
+      (effects (font (size 1.27 1.27)) (justify right) hide)
     )
   )
@@
     )
   )
-  (global_label "RGB MCU" (shape input) (at 103.505 27.305 0) (fields_autoplaced)
-    (effects (font (size 1.27 1.27)) (justify left))
-    (property "Intersheetrefs" "${INTERSHEET_REFS}" (at 115.0347 27.305 0)
-      (effects (font (size 1.27 1.27)) (justify left) hide)
-    )
+  (global_label "RGB MCU" (shape input) (at 103.505 45.085 0) (fields_autoplaced)
+    (effects (font (size 1.27 1.27)) (justify left))
+    (property "Intersheetrefs" "${INTERSHEET_REFS}" (at 115.0347 45.085 0)
+      (effects (font (size 1.27 1.27)) (justify left) hide)
+    )

Commit message: Revert "changed rgb pin for better software hardware compatibility & fresh production files"
This reverts commit 76bec49334091c1669f5db898bd2653646399791.
Connections:
- net RGB MCU: now also U1.11 (PA1); no longer U1.29 (PA8)
- net col0: now also U1.10 (PA0); no longer U1.11 (PA1)
- net rD: now also U1.29 (PA8); no longer U1.28 (PB15)
Changed lines of the file:
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@@
   (no_connect (at 70.485 85.725))
   (no_connect (at 217.805 74.93))
+  (no_connect (at 70.485 90.805))
   (no_connect (at 70.485 47.625))
-  (no_connect (at 103.505 24.765))
   (no_connect (at 70.485 88.265))
   (no_connect (at 70.485 83.185))
@@
     )
   )
-  (global_label "col0" (shape input) (at 103.505 27.305 0) (fields_autoplaced)
-    (effects (font (size 1.27 1.27)) (justify left))
-    (property "Intersheetrefs" "${INTERSHEET_REFS}" (at 110.5231 27.305 0)
+  (global_label "col0" (shape input) (at 103.505 24.765 0) (fields_autoplaced)
+    (effects (font (size 1.27 1.27)) (justify left))
+    (property "Intersheetrefs" "${INTERSHEET_REFS}" (at 110.5231 24.765 0)
       (effects (font (size 1.27 1.27)) (justify left) hide)
     )
@@
     )
   )
-  (global_label "rD" (shape input) (at 70.485 90.805 180) (fields_autoplaced)
-    (effects (font (size 1.27 1.27)) (justify right))
-    (property "Intersheetrefs" "${INTERSHEET_REFS}" (at 65.523 90.805 0)
-      (effects (font (size 1.27 1.27)) (justify right) hide)
+  (global_label "rD" (shape input) (at 103.505 45.085 0) (fields_autoplaced)
+    (effects (font (size 1.27 1.27)) (justify left))
+    (property "Intersheetrefs" "${INTERSHEET_REFS}" (at 108.467 45.085 0)
+      (effects (font (size 1.27 1.27)) (justify left) hide)
     )
   )
@@
     )
   )
-  (global_label "RGB MCU" (shape input) (at 103.505 45.085 0) (fields_autoplaced)
-    (effects (font (size 1.27 1.27)) (justify left))
-    (property "Intersheetrefs" "${INTERSHEET_REFS}" (at 115.0347 45.085 0)
-      (effects (font (size 1.27 1.27)) (justify left) hide)
-    )
+  (global_label "RGB MCU" (shape input) (at 103.505 27.305 0) (fields_autoplaced)
+    (effects (font (size 1.27 1.27)) (justify left))
+    (property "Intersheetrefs" "${INTERSHEET_REFS}" (at 115.0347 27.305 0)
+      (effects (font (size 1.27 1.27)) (justify left) hide)
+    )
